File: Hardware/AltusCharger/AltusCharger.kicad_sch (KiCad schematic)
At the start: 66 parts, among them J1 Conn_01x02_Socket, J2 Conn_01x02_Socket, J3 USB_C_Receptacle_USB2.0_16P, J4 Conn_01x02_Socket, J5 Conn_01x02_Socket, J6 Conn_01x02_Socket, J7 Conn_01x02_Socket, Q1 AO3401A, Q2 AO3400A, Q3 AO3400A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

Commit message: Mounting holes for schematic
Parts:
- added H1, H2, H3, H4: MountingHole, MountingHole:MountingHole_3.2mm_M3, symbol Mechanical:MountingHole
